File: extension/Revision History.kicad_sch (KiCad schematic)
At the start: 0 parts

Commit message: Task: Working on revision 1.0.0
Signed-off-by: Daniel Kampert <DanielKampert@kampis-elektroecke.de>
Changed lines of the file:
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@@
 		)
 	)
-	(text_box "${RELEASE_BODY_1.3.0}"
+	(text_box "${RELEASE_BODY_1.0.0}"
 		(exclude_from_sim no)
 		(at 22.86 35.56 0)
@@
 		)
 	)
-	(text_box "${RELEASE_TITLE_1.3.0}"
+	(text_box "${RELEASE_TITLE_1.0.0}"
 		(exclude_from_sim no)
 		(at 20.32 31.75 0)
