File: extension/Main.kicad_sch (KiCad schematic)
At the start: 38 parts, among them IC501 DA7212-01UM2, IC502 MAX32664, IC503 MAX86141, IC504 LIS2DS12, X501 MB1, X502 MB2, Y501 32kHz

Commit message: First version of the Layout and the Schematics is done
Parts:
- removed R501: 10k, Resistor_SMD:R_0201_0603Metric, symbol Device:R_Small
- C515: manf TAIYO YUDEN -> (none); manf# AMK105CBJ106MV-F -> (none); mouser# 963-AMK105CBJ106MV-F -> (none)
- C517: manf KYOCERA AVX -> (none); manf# 02016W105MAT2A -> (none); mouser# 581-02016W105MAT2A -> (none)
- C518: manf# C0402C104K4RAC7411 -> C0201C104K4RAC7411; mouser# 80-C0402C104K4R7411 -> 80-C0201C104K4RAC7411
- C520: manf TAIYO YUDEN -> (none); manf# MEASP105CC6226MF1A01 -> (none); mouser# 963-MEASP105CC62261A -> (none)
Connections:
- net GND: now also X502.1 (Pin_1); no longer X502.13 (Pin_13)
- net SCL: now also X502.10 (Pin_10); no longer X502.12 (Pin_12)
- net SDA: now also X502.8 (Pin_8); no longer X502.10 (Pin_10)
- net STATUS: now also X502.12 (Pin_12); no longer X502.14 (Pin_14)
- net VSYS: now also X502.2 (Pin_2); no longer X502.1 (Pin_1)
- net ~{RESET_{HR}}: now also X502.14 (Pin_14); no longer X502.11 (Pin_11)
- net at D502.1 (K): now also IC503.D5 (PD1-IN); no longer IC503.D4 (PD2-IN)
- net at D501.1 (K): now also IC503.D4 (PD2-IN); no longer IC503.D5 (PD1-IN)
- no-connect marks 24 -> 19
Other:
- moved on the sheet: D501, D502
