File: extension/ZSWatch-Extension.kicad_sch (KiCad schematic)
At the start: 0 parts

Commit message: Task: Working on revision 1.0.0
Signed-off-by: Daniel Kampert <DanielKampert@kampis-elektroecke.de>
Other:
- added sheet Power - Topology (Power - Topology.kicad_sch)
- title: Heartrate-HW -> Extension-HW
Changed lines of the file:
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@@
 	(paper "A3")
 	(title_block
-		(title "Heartrate-HW")
+		(title "Extension-HW")
 		(date "2025-07-13")
 		(rev "${REVISION}")
@@
 				)
 			)
-			(project "ZSWatch-Heartrate"
+			(project "ZSWatch-Extension"
 				(path "/d5742f03-3b1a-42e5-a384-018bd4b919aa"
 					(page "5")
@@
 				)
 			)
-			(project "ZSWatch-Heartrate"
+			(project "ZSWatch-Extension"
 				(path "/d5742f03-3b1a-42e5-a384-018bd4b919aa"
 					(page "2")
@@
 			(color 0 0 0 0.0000)
 		)
-		(property "Sheetname" "Project Architecture"
+		(property "Sheetname" "Power - Topology"
 			(at 306.07 313.9309 0)
 			(effects
@@
 			)
 		)
-		(property "Sheetfile" "Project Architecture.kicad_sch"
+		(property "Sheetfile" "Power - Topology.kicad_sch"
 			(at 307.34 316.23 0)
 			(effects
@@
 		)
 		(instances
+			(project "ZSWatch-Extension"
+				(path "/d5742f03-3b1a-42e5-a384-018bd4b919aa"
+					(page "3")
+				)
+			)
+		)
+	)
+	(sheet
+		(at 346.71 314.96)
+		(size 35.56 5.08)
+		(exclude_from_sim no)
+		(in_bom yes)
+		(on_board yes)
+		(dnp no)
+		(stroke
+			(width 0.1524)
+			(type solid)
+		)
+		(fill
+			(color 0 0 0 0.0000)
+		)
+		(property "Sheetname" "Project Architecture"
+			(at 346.71 313.9309 0)
+			(effects
+				(font
+					(face "Times New Roman")
+					(size 1.905 1.905)
+					(bold yes)
+					(color 0 0 0 1)
+				)
+				(justify left bottom)
+			)
+		)
+		(property "Sheetfile" "Project Architecture.kicad_sch"
+			(at 347.98 316.23 0)
+			(effects
+				(font
+					(face "Arial")
+					(size 1.27 1.27)
+				)
+				(justify left top)
+			)
+		)
+		(instances
 			(project "KDT_Hierarchical_KiBot"
 				(path "/f9e05184-c88b-4a88-ae9c-ab2bdb32be7c"
@@
 				)
 			)
-			(project "ZSWatch-Heartrate"
+			(project "ZSWatch-Extension"
 				(path "/d5742f03-3b1a-42e5-a384-018bd4b919aa"
 					(page "3")
