File: extension/Audio.kicad_sch (KiCad schematic)
At the start: 15 parts, among them IC601 DA7212-01UM2

Commit message: Change connector layout to simplify routing on the watch PCB
Other:
- title: Heartrate-DevKit -> Audio
Changed lines of the file:
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@@
 	(paper "A4")
 	(title_block
-		(title "Heartrate-DevKit")
+		(title "Audio")
 		(date "2025-07-13")
 		(rev "${REVISION}")
