File: extension/Connectors.kicad_sch (KiCad schematic)
At the start: 2 parts, among them X701 MB2, X702 MB1

Commit message: Bug: Issue #4
- Sheet titles missing

Closes: #4

Signed-off-by: Daniel Kampert <DanielKampert@kampis-elektroecke.de>
Other:
- title: (none) -> Connectors
Changed lines of the file:
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@@
 	(paper "A4")
 	(title_block
+		(title "Connectors")
 		(date "2025-07-13")
 		(rev "${REVISION}")
