File: extension/Connectors.kicad_sch (KiCad schematic)
At the start: 2 parts, among them X701 MB2, X702 MB1

Commit message: Add power rail test points and mounting orientation arrow
Parts:
- added TP1: 1V8_PA, TestPoint:TestPoint_Pad_D1.0mm, symbol Connector:TestPoint
- added TP2: 1V8_HR, TestPoint:TestPoint_Pad_D1.0mm, symbol Connector:TestPoint
- added TP3: VSYS, TestPoint:TestPoint_Pad_D1.0mm, symbol Connector:TestPoint
Connections:
- net +1V8_HR: now also TP2.1
- net +1V8_PA: now also TP1.1
- net VSYS: now also TP3.1

Commit message: Bug: Issue #4
- Sheet titles missing

Closes: #4

Signed-off-by: Daniel Kampert <DanielKampert@kampis-elektroecke.de>
Other:
- title: (none) -> Connectors
Changed lines of the file:
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@@
 	(paper "A4")
 	(title_block
+		(title "Connectors")
 		(date "2025-07-13")
 		(rev "${REVISION}")
