File: extension/ZSWatch-Extension.kicad_pcb (KiCad board)
At the start: 4 copper layers, 16.8 x 16.8 mm, 40 parts, among them IC501 MAX32664, IC502 LIS2DS12, IC503 MAX86141, IC601 DA7212-01UM2, X701 MB2, X702 MB1, Y501 32kHz

Commit message: Preserve test-point labels and validate combined release layout
Parts:
- renumbered PA to TP1, HR to TP2, V to TP3
Other:
- board text added: "HR"
- board text added: "PA"
- board text added: "V"
Changed lines of the file:
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@@
 		(descr "SMD pad as test Point, diameter 1.0mm")
 		(tags "test point SMD pad")
-		(property "Reference" "PA"
+		(property "Reference" "TP1"
 			(at -2.1 0.8 0)
 			(layer "B.SilkS")
+			(hide yes)
 			(effects
 				(font
@@
 		(descr "SMD pad as test Point, diameter 1.0mm")
 		(tags "test point SMD pad")
-		(property "Reference" "HR"
+		(property "Reference" "TP2"
 			(at 0 1.448 0)
 			(layer "B.SilkS")
+			(hide yes)
 			(effects
 				(font
@@
 		(descr "SMD pad as test Point, diameter 1.0mm")
 		(tags "test point SMD pad")
-		(property "Reference" "V"
+		(property "Reference" "TP3"
 			(at -1.2 -0.1 0)
 			(layer "B.SilkS")
+			(hide yes)
 			(effects
 				(font
@@
 		(net 69)
 	)
+	(gr_text "PA"
+		(at 208.2 156.1 0)
+		(layer "B.SilkS")
+		(effects
+			(font
+				(size 1 1)
+				(thickness 0.15)
+			)
+			(justify mirror)
+		)
+	)
+	(gr_text "HR"
+		(at 199 152.652 0)
+		(layer "B.SilkS")
+		(effects
+			(font
+				(size 1 1)
+				(thickness 0.15)
+			)
+			(justify mirror)
+		)
+	)
+	(gr_text "V"
+		(at 199.5 148.5 0)
+		(layer "B.SilkS")
+		(effects
+			(font
+				(size 1 1)
+				(thickness 0.15)
+			)
+			(justify mirror)
+		)
+	)
 )
